File: protoflow/DSO_1draft.kicad_pcb (KiCad board)
At the start: 2 copper layers, 90 x 69 mm, 130 parts, among them J1 Conn_01x05, J2 Conn_Coaxial, J3 Conn_Coaxial, J4 Conn_Coaxial, J5 Conn_Coaxial, J7 USB_A_Stacked, J8 Conn_01x20, J9 Conn_01x20, SW1 SW_SPDT, SW2 SW_SPDT, SW3 SW_SPDT, SW4 SW_SPDT, SW5 SW_SPDT, U1 ADG708BRUZ, U2 ADG708BRUZ, U3 STM32G431C6Tx

Commit message: added confirmed pcb
Parts:
- C1, C42: moved to F.Cu
- C10, C11, C12, C13, C14, C15, C16, C17, C18, C19, C36, C37, C38, C39, C4, C5, C8, C9, R10, R11, R12, R13, R3, R4, R47, R5, R6, R7, R8, R9, digildo1, pwmoppamp1: moved to B.Cu
- moved R52 213.7 mm to (244.9, 38.3), turned to 90 degrees
- moved R51 205.6 mm to (237.3, 38.5), turned to 90 degrees
- moved C30 198.3 mm to (222.0, 127.4)
- moved R50 197.9 mm to (229.8, 38.5), turned to 90 degrees
- moved C29 186.7 mm to (210.9, 127.5), turned to 180 degrees
- moved R21 168.5 mm to (228.4, 145.2), turned to 90 degrees
- moved R15 156.5 mm to (220.9, 150.4), turned to 90 degrees
- moved R45 154.7 mm to (216.6, 127.4)
- moved R43 151.3 mm to (219.8, 137.1)
- moved D6 148.6 mm to (248.7, 38.4)
- moved R44 147.5 mm to (212.3, 131.8), turned to 90 degrees
- moved R42 145.1 mm to (214.4, 137.1)
- moved D5 144.2 mm to (240.7, 38.6)
- moved U2 140.8 mm to (232.1, 46.5)
- moved D4 140.1 mm to (233.1, 38.5)
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Routing:
- net /5v: track 14.0 -> 68.8 mm
- net Net-(J7-Shield): track 0.00 -> 44.3 mm
- net GND: track 0.00 -> 28.8 mm
- net /pwmopout4: track 0.00 -> 13.4 mm, vias 0 -> 2
- net Net-(C16-Pad1): track 0.00 -> 12.3 mm
- net /funcout1: track 0.00 -> 12.1 mm
- net /B2: track 0.00 -> 12.0 mm
- net /S6B: track 0.00 -> 11.2 mm
- net /funcout2: track 0.00 -> 10.8 mm
- net /-5v: track 10.7 -> 0.00 mm
- net /pwmopout3: track 0.00 -> 10.1 mm
- net /S4B: track 0.00 -> 9.85 mm
- net /S3B: track 0.00 -> 9.82 mm
- net Net-(C19-Pad1): track 0.00 -> 9.77 mm
- net /S5B: track 0.00 -> 9.50 mm
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Other:
- board size 90 x 69 mm -> 99.9 x 70 mm
- board text added: "See about This later ->"

Commit message: moved neccesary things
Parts:
- R17, R18, R19, R20: moved to B.Cu
- moved J1 170.9 mm to (167.8, 146.2)
- moved C31 136.1 mm to (135.0, 106.0)
- moved C32 135.9 mm to (146.0, 123.0)
- moved R49 130.6 mm to (116.0, 138.0)
- moved R38 124.0 mm to (142.0, 97.0)
- moved SW2 121.5 mm to (114.2, 123.5)
- moved D3 116.1 mm to (113.0, 137.0)
- moved D1 109.8 mm to (132.8, 87.2), turned to -90 degrees
- moved D4 104.4 mm to (150.9, 102.8)
- moved D6 104.4 mm to (166.5, 102.7)
- moved U2 104.4 mm to (149.9, 110.8)
- moved D5 104.4 mm to (158.5, 102.9)
- moved R30 104.4 mm to (144.0, 108.9)
- moved R32 104.4 mm to (138.2, 112.7)
- moved R34 104.4 mm to (146.6, 117.3)
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Routing:
- net GND: track 28.8 -> 121.7 mm
- net /pwmout4: track 6.55 -> 86.1 mm
- net /pwmout3: track 7.86 -> 68.6 mm
- net /5v: track 68.8 -> 50.3 mm
- net Net-(J7-D1-): track 17.2 -> 0.00 mm
- net /pwmopout4: track 13.4 -> 27.7 mm, vias 2 -> 0
- net Net-(funcopamp1-1IN-): track 0.00 -> 12.4 mm
- net /funcout2: track 10.8 -> 19.5 mm
- net Net-(funcopamp1-2IN-): track 0.00 -> 8.14 mm
- net Net-(C8-Pad1): track 6.55 -> 12.6 mm
- net /3v3: track 9.48 -> 4.20 mm
- net Net-(C10-Pad1): track 11.4 -> 15.4 mm
- net /funcout1: track 12.1 -> 15.8 mm
- net Net-(D3-A): track 0.00 -> 3.35 mm
- net Net-(C11-Pad1): track 6.43 -> 9.44 mm
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
Commit message: completed pcb design
Parts:
- C13, C14, C15, C18, C36, C38, R47: moved to F.Cu
- C21, C26, C32, C33, C34, C40, C41, R21, R22, R25, R26, R27, R29, R31, R33, R34, R37, R40, R43, R45, R48: moved to B.Cu
- moved R52 52.0 mm to (122.9, 136.0), turned to 0 degrees
- moved D6 51.1 mm to (127.8, 136.0), turned to 180 degrees
- moved C40 46.6 mm to (128.2, 128.7), turned to -90 degrees
- moved R51 43.8 mm to (122.9, 132.6), turned to 0 degrees
- moved D5 42.7 mm to (127.8, 132.6), turned to 180 degrees
- moved R55 39.0 mm to (112.0, 136.0), turned to 0 degrees
- moved D9 38.6 mm to (116.9, 136.0), turned to 180 degrees
- moved C41 37.4 mm to (141.0, 140.0), turned to 180 degrees
- moved R50 36.2 mm to (122.9, 129.2), turned to 0 degrees
- moved D4 35.1 mm to (127.8, 129.2), turned to 180 degrees
- moved R54 34.2 mm to (112.0, 132.6), turned to 0 degrees
- moved D8 34.2 mm to (116.9, 132.6), turned to 180 degrees
- moved C21 33.6 mm to (133.8, 137.6), turned to -90 degrees
- moved D7 31.0 mm to (116.9, 129.2), turned to 180 degrees
- moved R53 30.6 mm to (112.0, 129.2), turned to 0 degrees
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Routing:
- net /PG10_NRST: track 0.00 -> 205.5 mm, vias 0 -> 4
- net /A1: track 5.90 -> 176.3 mm, vias 0 -> 8
- net /3v3: track 4.20 -> 167.5 mm, vias 0 -> 12
- net /B2: track 12.0 -> 164.3 mm, vias 0 -> 4
- net /D+: track 0.00 -> 142.7 mm, vias 0 -> 4
- net /A2: track 11.9 -> 146.6 mm, vias 0 -> 4
- net /S1B: track 5.46 -> 139.8 mm, vias 0 -> 4
- net /OP4_OUT: track 6.41 -> 140.1 mm, vias 0 -> 3
- net /PA0_ADC_IN1: track 0.00 -> 128.3 mm, vias 0 -> 8
- net /3v3_digi: track 0.00 -> 125.2 mm, vias 0 -> 9
- net /S0: track 7.24 -> 131.8 mm, vias 1 -> 11
- net /DAC2: track 0.00 -> 113.2 mm, vias 0 -> 8
- net /D-: track 0.00 -> 104.5 mm, vias 0 -> 4
- net /EOP-: track 0.00 -> 98.6 mm, vias 0 -> 4
- net /EOP_OUT: track 0.00 -> 96.3 mm, vias 0 -> 1
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- added copper zone on B.Cu, net GND
- added copper zone on F.Cu, net GND
Other:
- board size 99.9 x 70 mm -> 99.9 x 77.2 mm

Commit message: your commit message
Routing:
- net GND: track 57.2 -> 76.3 mm, vias 56 -> 58
Changed lines of the file:
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@@
+	)
+	(segment
+		(start 136.212 108.1)
+		(end 138.312 108.1)
+		(width 0.3)
+		(layer "F.Cu")
+		(net "GND")
 	)
 	(segment
@@
 	)
 	(segment
+		(start 119.45 136)
+		(end 118.85 135.2)
+		(width 0.3)
+		(layer "F.Cu")
+		(net "GND")
+	)
+	(segment
+		(start 160.35 111.537)
+		(end 161.55 112.537)
+		(width 0.3)
+		(layer "F.Cu")
+		(net "GND")
+	)
+	(segment
 		(start 148.3 110)
 		(end 148.8 110.5)
@@
 	)
 	(segment
+		(start 136.212 108.1)
+		(end 137.412 108.1)
+		(width 0.3)
+		(layer "F.Cu")
+		(net "GND")
+	)
+	(segment
 		(start 148.8 110.5)
 		(end 149.5 110.5)
@@
 	)
 	(segment
+		(start 160.35 111.537)
+		(end 160.65 112.537)
+		(width 0.3)
+		(layer "F.Cu")
+		(net "GND")
+	)
+	(segment
 		(start 149.5 110.5)
 		(end 149.55 110.55)
@@
 	)
 	(via
-		(at 134.787 125.7)
+		(at 134.787 125.3)
 		(size 0.6)
 		(drill 0.3)
@@
 	)
 	(via
-		(at 118.85 135.2)
+		(at 119.45 136)
 		(size 0.5)
 		(drill 0.3)
@@
 	)
 	(via
-		(at 133 139.4)
+		(at 134.8 137.1)
 		(size 0.5)
 		(drill 0.3)
@@
 	)
 	(via
-		(at 160.65 112.537)
+		(at 160.35 111.537)
 		(size 0.6)
 		(drill 0.3)
@@
 	)
 	(via
-		(at 138.312 108.1)
+		(at 136.212 108.1)
 		(size 0.6)
 		(drill 0.3)
@@
 	)
 	(via
+		(at 127.54 136.84)
+		(size 0.6)
+		(drill 0.3)
+		(layers "F.Cu" "B.Cu")
+		(net "GND")
+	)
+	(via
 		(at 133.025 137.125)
 		(size 0.6)
@@
 	)
 	(via
-		(at 149.951 108.364)
-		(size 0.6)
-		(drill 0.3)
-		(layers "F.Cu" "B.Cu")
-		(net "GND")
-	)
-	(via
-		(at 134.386 139.749)
+		(at 149.451 108.364)
+		(size 0.6)
+		(drill 0.3)
+		(layers "F.Cu" "B.Cu")
+		(net "GND")
+	)
+	(via
+		(at 135.286 136.649)
 		(size 0.6)
 		(drill 0.3)
@@
 	)
 	(via
-		(at 127.65 134.9)
+		(at 127.65 133.7)
 		(size 0.5)
 		(drill 0.3)
@@
 	)
 	(via
+		(at 135.06 138.24)
+		(size 0.6)
+		(drill 0.3)
+		(layers "F.Cu" "B.Cu")
+		(net "GND")
+	)
+	(via
 		(at 158.4 138.4)
 		(size 0.5)
@@
 	)
 	(via
-		(at 140.7 122.938)
+		(at 140.6 122.638)
 		(size 0.6)
 		(drill 0.3)
@@
 	)
 	(segment
+		(start 127.65 133.7)
+		(end 127.65 134.9)
+		(width 0.3)
+		(layer "B.Cu")
+		(net "GND")
+	)
+	(segment
 		(start 116.6 118.95)
 		(end 116.6 120.05)
@@
 	)
 	(segment
+		(start 134.787 125.3)
+		(end 134.787 126.7)
+		(width 0.3)
+		(layer "B.Cu")
+		(net "GND")
+	)
+	(segment
 		(start 118.85 135.2)
 		(end 118.85 133.65)
@@
 	)
 	(segment
+		(start 140.6 122.638)
+		(end 140.7 122.938)
+		(width 0.3)
+		(layer "B.Cu")
+		(net "GND")
+	)
+	(segment
 		(start 151.275 126.775)
 		(end 151.275 128.525)
@@
 	)
 	(segment
+		(start 135.286 136.649)
+		(end 134.386 139.749)
+		(width 0.3)
+		(layer "B.Cu")
+		(net "GND")
+	)
+	(segment
 		(start 142.4 138.359744)
 		(end 142.4 136)
@@
 	)
 	(segment
+		(start 134.8 137.1)
+		(end 133 139.4)
+		(width 0.3)
+		(layer "B.Cu")
+		(net "GND")
+	)
+	(segment
 		(start 127.9125 135.35)
 		(end 128.575 135.35)
@@
 	)
 	(segment
+		(start 134.787 125.3)
+		(end 134.787 125.7)
+		(width 0.3)
+		(layer "B.Cu")
+		(net "GND")
+	)
+	(segment
 		(start 139.4375 140)
 		(end 138.7375 139.3)
@@
 	)
 	(segment
+		(start 119.45 136)
+		(end 118.85 135.2)
+		(width 0.3)
+		(layer "B.Cu")
+		(net "GND")
+	)
+	(segment
 		(start 133.75 139.1125)
 		(end 134.386 139.749)
@@
 	)
 	(segment
+		(start 140.6 122.638)
+		(end 140.7 123.838)
+		(width 0.3)
+		(layer "B.Cu")
+		(net "GND")
+	)
+	(segment
 		(start 116.65 118.9)
 		(end 116.6 118.95)
@@
 		(layer "B.Cu")
 		(net "GND")
+	)
+	(segment
+		(start 149.451 108.364)
+		(end 149.951 108.364)
+		(width 0.3)
+		(layer "B.Cu")
+		(net "GND")

Commit message: final output
Parts:
- removed SW4, SW5: SW_SPDT, Slide_switch:SS-12F17_1P2T
- moved R56 47.5 mm to (171.9, 142.2)
- moved C11 37.5 mm to (178.0, 115.0)
- moved C24 35.3 mm to (144.0, 109.0), turned to 180 degrees
- moved J9 34.9 mm to (103.1, 152.5)
- moved C23 33.1 mm to (151.5, 103.2), turned to 90 degrees
- moved R5 32.6 mm to (173.6, 115.4), turned to 0 degrees
- moved C29 31.7 mm to (175.6, 111.2), turned to 0 degrees
- moved R6 30.7 mm to (177.6, 121.1), turned to -90 degrees
- moved R21 30.4 mm to (149.8, 106.4), turned to -90 degrees
- moved C16 28.9 mm to (175.2, 135.4), turned to 90 degrees
- moved R41 28.5 mm to (164.6, 103.2), turned to -90 degrees
- moved C26 28.4 mm to (164.5, 103.2), turned to 90 degrees
- moved C37 28.3 mm to (176.4, 129.7), turned to 180 degrees
- moved R7 28.0 mm to (176.4, 126.6), turned to 180 degrees
- moved C28 27.9 mm to (146.8, 116.0)
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Connections:
- J7 pad 2: Net-(J7-D1-) -> unconnected-(J7-D1--Pad2)
- J7 pad 3: Net-(J7-D1+) -> unconnected-(J7-D1+-Pad3)
- J7 pad 6: Net-(J7-D2-) -> /D-
- J7 pad 7: Net-(J7-D2+) -> /D+
- J8 pad 1: /PF0 -> /PB11_TM2_4
- J8 pad 10: /PA9 -> /PF0
- J8 pad 11: /PA10 -> /PC15
- J8 pad 12: /EOP+ -> /PC14
- J8 pad 13: /EOP- -> /PC13
- J8 pad 14: /EOP_OUT -> /EOP+
- J8 pad 15: /PB8 -> /EOP-
- J8 pad 16: /PG10_NRST -> /EOP_OUT
- J8 pad 2: /PF1 -> /PB10_TM2_3
- J8 pad 3: /PC13 -> /PA0_ADC_IN1
- J8 pad 4: /PC14 -> /B0
- J8 pad 5: /PC15 -> /PA7
- J8 pad 6: /PB12 -> /DAC2
- J8 pad 7: /PB14 -> /DAC1
- J8 pad 8: /PA7 -> /PG10_NRST
- J8 pad 9: /PA8 -> /PF1
- J9 pad 1: /PA0_ADC_IN1 -> /PB12
- J9 pad 10: /B1 -> /PB3_TM2_2
- J9 pad 11: /B2 -> /B1
- J9 pad 12: /A0 -> /B2
- J9 pad 13: /A1 -> /A0
- J9 pad 14: /A2 -> /A1
- J9 pad 15: /D- -> /PB8
- J9 pad 16: /D+ -> /A2
- J9 pad 2: /OP4_OUT -> /PB14
- J9 pad 3: /PB3_TM2_1 -> /OP4_OUT
- J9 pad 4: /PB3_TM2_2 -> /PA8
- J9 pad 5: /PB3_TM2_3 -> /PA9
- J9 pad 6: /PB3_TM2_4 -> /PA10
- J9 pad 7: /DAC1 -> /D-
- J9 pad 8: /DAC2 -> /D+
- J9 pad 9: /B0 -> /PA15_TM2_1
- R11 pad 1: /PB3_TM2_4 -> /PB11_TM2_4
- R4 pad 1: /PB3_TM2_1 -> /PA15_TM2_1
- R8 pad 1: /PB3_TM2_3 -> /PB10_TM2_3
- anlgLDO1 pad 4: unconnected-(anlgLDO1-NC-Pad4) -> GND
- digildo1 pad 4: (no net) -> /3v3_digi
Routing:
- net GND: track 76.3 -> 631.7 mm, vias 58 -> 15
- net /PG10_NRST: track 205.5 -> 64.4 mm, vias 4 -> 1
- net /A1: track 176.3 -> 83.1 mm, vias 8 -> 5
- net /PB11_TM2_4: track 0.00 -> 89.3 mm, vias 0 -> 3
- net /D+: track 142.7 -> 68.7 mm, vias 4 -> 0
- net /PA15_TM2_1: track 0.00 -> 72.8 mm, vias 0 -> 3
- net /-5v: track 75.5 -> 147.2 mm
- net /PB3_TM2_3: track 69.7 -> 0.00 mm, vias 4 -> 0
- net /PB3_TM2_2: track 38.3 -> 106.9 mm, vias 2 -> 7
- net /PC13: track 84.3 -> 23.4 mm, vias 2 -> 1
- net /B2: track 164.3 -> 103.7 mm, vias 4 -> 5
- net /A2: track 146.6 -> 86.0 mm, vias 4 -> 1
- net /PB10_TM2_3: track 0.00 -> 57.5 mm, vias 0 -> 2
- net /EOP_OUT: track 96.3 -> 45.2 mm, vias 1 -> 5
- net /OP4_OUT: track 140.1 -> 89.8 mm
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- added copper zone on F.Cu, net /3v3
- added copper zone on F.Cu, net /5v
- removed copper zone on F.Cu, net GND
Other:
- board size 99.9 x 77.2 mm -> 98 x 78.9 mm
- board text removed: "See about This later ->"
