File: protoflow/DSO_1draft.kicad_sch (KiCad schematic)
At the start: 130 parts, among them J1 Conn_01x05, J2 Conn_Coaxial, J3 Conn_Coaxial, J4 Conn_Coaxial, J5 Conn_Coaxial, J7 USB_A_Stacked, J8 Conn_01x20, J9 Conn_01x20, SW1 SW_SPDT, SW2 SW_SPDT, SW3 SW_SPDT, SW4 SW_SPDT, SW5 SW_SPDT, U1 ADG708BRUZ, U2 ADG708BRUZ, U3 STM32G431C6Tx

Commit message: moved neccesary things
Other:
- moved on the sheet: C10, C11, C12, C13, C14, C15, C16, C17, C18, C19, C36, C37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

Commit message: updated according to pcb
Parts:
- removed SW4, SW5: SW_SPDT, Slide_switch:SS-12F17_1P2T, symbol Switch:SW_SPDT
Connections:
- net -5v: no longer J8.19 (Pin_19)
- net 3v3_digi: now also digildo1.4 (Heatsink); no longer J8.18 (Pin_18)
- net 5v: no longer J8.17 (Pin_17)
- net A0: no longer J9.12 (Pin_12)
- net A1: no longer J9.13 (Pin_13)
- net A2: no longer J9.14 (Pin_14)
- net B0: no longer J9.9 (Pin_9)
- net B1: no longer J9.10 (Pin_10)
- net B2: no longer J9.11 (Pin_11)
- net D+: now also J7.7 (D2+); no longer J9.16 (Pin_16)
- net D-: now also J7.6 (D2-); no longer J9.15 (Pin_15)
- net DAC1: no longer J9.7 (Pin_7)
- net DAC2: no longer J9.8 (Pin_8)
- net EOP+: no longer J8.12 (Pin_12)
- net EOP-: no longer J8.13 (Pin_13)
- net EOP_OUT: no longer J8.14 (Pin_14)
- net GND: no longer J8.20 (Pin_20)
- net OP4_OUT: no longer J9.2 (Pin_2)
- net PA0_ADC_IN1: no longer J9.1 (Pin_1)
- net PA10: no longer J8.11 (Pin_11)
- net PA15_TM2_1: now also R4.1
- net PA7: no longer J8.8 (Pin_8)
- net PA8: no longer J8.9 (Pin_9)
- net PA9: no longer J8.10 (Pin_10)
- net PB10_TM2_3: now also R8.1
- net PB11_TM2_4: now also R11.1
- net PB12: no longer J8.6 (Pin_6)
- net PB14: no longer J8.7 (Pin_7)
- net PB3_TM2_2: no longer J9.4 (Pin_4)
- net PB8: no longer J8.15 (Pin_15)
- net PC13: no longer J8.3 (Pin_3)
- net PC14: no longer J8.4 (Pin_4)
- net PC15: no longer J8.5 (Pin_5)
- net PF0: no longer J8.1 (Pin_1)
- net PF1: no longer J8.2 (Pin_2)
- net PG10_NRST: no longer J8.16 (Pin_16)
- net S0: no longer J9.18 (Pin_18)
- net S1B: no longer J9.17 (Pin_17)
- net PB3_TM2_1: no longer names the net of J9.3 (Pin_3)
- net PB3_TM2_1: no longer R4.1
- net PB3_TM2_3: no longer names the net of J9.5 (Pin_5)
- net PB3_TM2_3: no longer R8.1
- net PB3_TM2_4: no longer names the net of J9.6 (Pin_6)
- net PB3_TM2_4: no longer R11.1
- no-connect marks 4 -> 6

Commit message: final output
Connections:
- net -5v: now also J8.19 (Pin_19)
- net 3v3_digi: now also J8.18 (Pin_18)
- net 5v: now also J8.17 (Pin_17)
- net A0: now also J9.13 (Pin_13)
- net A1: now also J9.14 (Pin_14)
- net A2: now also J9.16 (Pin_16)
- net B0: now also J8.4 (Pin_4)
- net B1: now also J9.11 (Pin_11)
- net B2: now also J9.12 (Pin_12)
- net D+: now also J9.8 (Pin_8)
- net D-: now also J9.7 (Pin_7)
- net DAC1: now also J8.7 (Pin_7)
- net DAC2: now also J8.6 (Pin_6)
- net EOP+: now also J8.14 (Pin_14)
- net EOP-: now also J8.15 (Pin_15)
- net EOP_OUT: now also J8.16 (Pin_16)
- net GND: now also J8.20 (Pin_20), anlgLDO1.4 (NC)
- net OP4_OUT: now also J9.3 (Pin_3)
- net PA0_ADC_IN1: now also J8.3 (Pin_3)
- net PA10: now also J9.6 (Pin_6)
- net PA15_TM2_1: now also J9.9 (Pin_9)
- net PA7: now also J8.5 (Pin_5)
- net PA8: now also J9.4 (Pin_4)
- net PA9: now also J9.5 (Pin_5)
- net PB10_TM2_3: now also J8.2 (Pin_2)
- net PB11_TM2_4: now also J8.1 (Pin_1)
- net PB12: now also J9.1 (Pin_1)
- net PB14: now also J9.2 (Pin_2)
- net PB3_TM2_2: now also J9.10 (Pin_10)
- net PB8: now also J9.15 (Pin_15)
- net PC13: now also J8.13 (Pin_13)
- net PC14: now also J8.12 (Pin_12)
- net PC15: now also J8.11 (Pin_11)
- net PF0: now also J8.10 (Pin_10)
- net PF1: now also J8.9 (Pin_9)
- net PG10_NRST: now also J8.8 (Pin_8)
- net S0: now also J9.18 (Pin_18)
- net S1B: now also J9.17 (Pin_17)
- no-connect marks 6 -> 5
Other:
- moved on the sheet: J8, J9
